File: .history/GBG_Motors.kicad_pcb (KiCad board)
At the start: 2 copper layers, 1 part

Commit message: Began layout phase
Parts:
- removed U1: ~, BTS7960:BTS7960
- added C601: 10uF, Capacitor_THT:C_Axial_L3.8mm_D2.6mm_P7.50mm_Horizontal, F.Cu at (241.2, 59.2)
- added C602: 10uF, Capacitor_THT:C_Axial_L3.8mm_D2.6mm_P7.50mm_Horizontal, F.Cu at (241.2, 63.4)
- added C701: 10uF, Capacitor_THT:C_Axial_L3.8mm_D2.6mm_P7.50mm_Horizontal, F.Cu at (150.4, 56.3)
- added C702: 10uF, Capacitor_THT:C_Axial_L3.8mm_D2.6mm_P7.50mm_Horizontal, F.Cu at (176.3, 53.6)
- added J101: Input, Connector_PinHeader_2.54mm:PinHeader_1x06_P2.54mm_Vertical, F.Cu at (101.6, 50.8)
- added J102: Seeed XIAO L, Connector_PinHeader_2.54mm:PinHeader_1x07_P2.54mm_Vertical, F.Cu at (78.2, 101.6)
- added J103: Seeed XIAO R, Connector_PinHeader_2.54mm:PinHeader_1x07_P2.54mm_Vertical, F.Cu at (93.5, 101.6)
- added J104: Pin, Connector_PinHeader_2.54mm:PinHeader_1x02_P2.54mm_Vertical, F.Cu at (103.6, 40.6)
- added J105: Pout, Connector_PinHeader_2.54mm:PinHeader_1x02_P2.54mm_Vertical, F.Cu at (103.6, 71.1)
- added J601: Limit Switch, Connector_PinHeader_2.54mm:PinHeader_1x04_P2.54mm_Vertical, F.Cu at (263.5, 55.4)
- added J701: Limit Switch, Connector_PinHeader_2.54mm:PinHeader_1x04_P2.54mm_Vertical, F.Cu at (150.1, 34.5)
- added JP101: Input Vcc Sel, Jumper:SolderJumper-3_P1.3mm_Bridged12_RoundedPad1.0x1.5mm, F.Cu at (118.6, 15.7)
- added JP103: Regulator Bypass, Jumper:SolderJumper-2_P1.3mm_Bridged_RoundedPad1.0x1.5mm, B.Cu at (114.3, 43.2)
- added JP201: RA_skip, Jumper:SolderJumper-2_P1.3mm_Bridged_RoundedPad1.0x1.5mm, B.Cu at (111.9, 53.3)
- added JP301: RA_skip, Jumper:SolderJumper-2_P1.3mm_Bridged_RoundedPad1.0x1.5mm, B.Cu at (111.9, 55.9)
- added JP401: RA_skip, Jumper:SolderJumper-2_P1.3mm_Bridged_RoundedPad1.0x1.5mm, B.Cu at (111.9, 58.4)
- added JP501: RA_skip, Jumper:SolderJumper-2_P1.3mm_Bridged_RoundedPad1.0x1.5mm, B.Cu at (111.9, 61.0)
- added JP601: redirect, Jumper:SolderJumper-3_P1.3mm_Bridged12_RoundedPad1.0x1.5mm, F.Cu at (264.0, 47.2)
- added JP602: Limit Switch EN, Jumper:SolderJumper-2_P1.3mm_Bridged_RoundedPad1.0x1.5mm, F.Cu at (263.4, 67.1)
- added JP603: Timeout EN, Jumper:SolderJumper-3_P1.3mm_Bridged12_RoundedPad1.0x1.5mm, F.Cu at (264.0, 51.0)
- added JP701: Limit Switch EN, Jumper:SolderJumper-2_P1.3mm_Bridged_RoundedPad1.0x1.5mm, F.Cu at (202.4, 60.3)
- added JP702: redirect, Jumper:SolderJumper-3_P1.3mm_Bridged12_RoundedPad1.0x1.5mm, F.Cu at (145.8, 49.8)
- added JP703: Timeout EN, Jumper:SolderJumper-3_P1.3mm_Bridged12_RoundedPad1.0x1.5mm, F.Cu at (165.1, 61.7)
- added JP802: Redirect A, Jumper:SolderJumper-3_P1.3mm_Bridged12_RoundedPad1.0x1.5mm, F.Cu at (163.3, 115.8)
- added JP803: Redirect B, Jumper:SolderJumper-3_P1.3mm_Bridged12_RoundedPad1.0x1.5mm, F.Cu at (163.3, 119.7)
- added JP901: Redirect A, Jumper:SolderJumper-3_P1.3mm_Bridged12_RoundedPad1.0x1.5mm, F.Cu at (163.3, 106.2)
- added JP902: Redirect B, Jumper:SolderJumper-3_P1.3mm_Bridged12_RoundedPad1.0x1.5mm, F.Cu at (163.3, 110.0)
- added Q602: NPN, Package_TO_SOT_THT:TO-92_Wide, F.Cu at (241.2, 69.5)
- added Q701: NPN, Package_TO_SOT_THT:TO-92_Wide, F.Cu at (157.0, 51.1)
- added R201: RA, Resistor_THT:R_Axial_DIN0207_L6.3mm_D2.5mm_P7.62mm_Horizontal, F.Cu at (106.7, 53.3)
- added R202: RB, Resistor_THT:R_Axial_DIN0207_L6.3mm_D2.5mm_P7.62mm_Horizontal, F.Cu at (124.5, 53.3)
- added R301: RA, Resistor_THT:R_Axial_DIN0207_L6.3mm_D2.5mm_P7.62mm_Horizontal, F.Cu at (106.7, 55.9)
- added R302: RB, Resistor_THT:R_Axial_DIN0207_L6.3mm_D2.5mm_P7.62mm_Horizontal, F.Cu at (124.5, 55.9)
- added R401: RA, Resistor_THT:R_Axial_DIN0207_L6.3mm_D2.5mm_P7.62mm_Horizontal, F.Cu at (106.7, 58.4)
- added R402: RB, Resistor_THT:R_Axial_DIN0207_L6.3mm_D2.5mm_P7.62mm_Horizontal, F.Cu at (124.5, 58.4)
- added R501: RA, Resistor_THT:R_Axial_DIN0207_L6.3mm_D2.5mm_P7.62mm_Horizontal, F.Cu at (106.7, 61.0)
- added R502: RB, Resistor_THT:R_Axial_DIN0207_L6.3mm_D2.5mm_P7.62mm_Horizontal, F.Cu at (124.5, 61.0)
- added R601: R, Resistor_THT:R_Axial_DIN0207_L6.3mm_D2.5mm_P7.62mm_Horizontal, F.Cu at (252.0, 47.5)
- added R602: 10k, Resistor_THT:R_Axial_DIN0207_L6.3mm_D2.5mm_P7.62mm_Horizontal, F.Cu at (252.0, 51.5)
- added R603: 100k, Resistor_THT:R_Axial_DIN0207_L6.3mm_D2.5mm_P7.62mm_Horizontal, F.Cu at (252.0, 55.5)
- added R604: 100k, Resistor_THT:R_Axial_DIN0207_L6.3mm_D2.5mm_P7.62mm_Horizontal, F.Cu at (252.0, 59.6)
- added R605: 100k, Resistor_THT:R_Axial_DIN0207_L6.3mm_D2.5mm_P7.62mm_Horizontal, F.Cu at (252.0, 63.6)
- added R607: 10k, Resistor_THT:R_Axial_DIN0207_L6.3mm_D2.5mm_P7.62mm_Horizontal, F.Cu at (252.0, 67.7)
- added R701: R, Resistor_THT:R_Axial_DIN0207_L6.3mm_D2.5mm_P7.62mm_Horizontal, F.Cu at (191.0, 40.6)
- added R702: 10k, Resistor_THT:R_Axial_DIN0207_L6.3mm_D2.5mm_P7.62mm_Horizontal, F.Cu at (150.4, 53.6)
- added R703: 100k, Resistor_THT:R_Axial_DIN0207_L6.3mm_D2.5mm_P7.62mm_Horizontal, F.Cu at (191.0, 48.7)
- added R704: 100k, Resistor_THT:R_Axial_DIN0207_L6.3mm_D2.5mm_P7.62mm_Horizontal, F.Cu at (153.9, 63.8)
- added R705: 10k, Resistor_THT:R_Axial_DIN0207_L6.3mm_D2.5mm_P7.62mm_Horizontal, F.Cu at (157.5, 56.1)
- added R706: 100k, Resistor_THT:R_Axial_DIN0207_L6.3mm_D2.5mm_P7.62mm_Horizontal, F.Cu at (172.7, 46.0)
- added U101: JK Controller, BTS7960:BTS7960, F.Cu at (54.2, 48.0)
- added U102: HL Controller, BTS7960:BTS7960, F.Cu at (54.2, 99.1)
- added U103: R-78E5.0-0.5, Converter_DCDC:Converter_DCDC_RECOM_R-78E-0.5_THT, F.Cu at (109.6, 40.7)
- added U601: NE555P, Package_DIP:DIP-8_W7.62mm, F.Cu at (241.2, 47.5)
- added U701: NE555P, Package_DIP:DIP-8_W7.62mm, F.Cu at (161.3, 48.5)
Other:
- board text added: "401"
