File: .history/GBG_Motors.kicad_sch (KiCad schematic)
At the start: 1 part

Commit message: Began layout phase
Parts:
- removed U1: (no value), BTS7960:BTS7960, symbol BTS7960:BTS7960
- added J101: Input, Connector_PinHeader_2.54mm:PinHeader_1x06_P2.54mm_Vertical, symbol Connector:Conn_01x06_Pin
- added J102: Seeed XIAO L, Connector_PinHeader_2.54mm:PinHeader_1x07_P2.54mm_Vertical, symbol Connector:Conn_01x07_Pin
- added J103: Seeed XIAO R, Connector_PinHeader_2.54mm:PinHeader_1x07_P2.54mm_Vertical, symbol Connector:Conn_01x07_Pin
- added J104: Pin, Connector_PinHeader_2.54mm:PinHeader_1x02_P2.54mm_Vertical, symbol Connector:Conn_01x02_Pin
- added J105: Pout, Connector_PinHeader_2.54mm:PinHeader_1x02_P2.54mm_Vertical, symbol Connector:Conn_01x02_Pin
- added JP101: Input Vcc Sel, Jumper:SolderJumper-3_P1.3mm_Bridged12_RoundedPad1.0x1.5mm, symbol Jumper:SolderJumper_3_Bridged12
- added JP103: Regulator Bypass, Jumper:SolderJumper-2_P1.3mm_Bridged_RoundedPad1.0x1.5mm, symbol Jumper:Jumper_2_Open
- added U101: JK Controller, BTS7960:BTS7960, symbol BTS7960:BTS7960
- added U102: HL Controller, BTS7960:BTS7960, symbol BTS7960:BTS7960
- added U103: R-78E5.0-0.5, Converter_DCDC:Converter_DCDC_RECOM_R-78E-0.5_THT, symbol Converter_DCDC:R-78E5.0-0.5
Connections:
- new net +5V: J103.1 (Pin_1), JP101.1 (A), JP103.2 (B), U101.3 (R_EN), U101.4 (L_EN), U101.7 (Vcc), U102.3 (R_EN), U102.4 (L_EN), U102.7 (Vcc), U103.3 (OUT)
- new net GND: J101.6 (Pin_6), J103.2 (Pin_2), J104.2 (Pin_2), J105.2 (Pin_2), U101.8 (GND), U102.8 (GND), U103.2 (GND)
- new net H: J101.2 (Pin_2)
- new net HRi: J102.2 (Pin_2)
- new net HRo: J102.1 (Pin_1)
- new net Hc: U102.1 (RPWM)
- new net J: J101.3 (Pin_3)
- new net JRi: J102.4 (Pin_4)
- new net JRo: J102.3 (Pin_3)
- new net Jc: U101.2 (LPWM)
- new net K: J101.4 (Pin_4)
- new net KRi: J102.6 (Pin_6)
- new net KRo: J102.5 (Pin_5)
- new net Kc: U101.1 (RPWM)
- new net L: J101.5 (Pin_5)
- new net LRi: J103.5 (Pin_5)
- new net LRo: J103.6 (Pin_6)
- new net Lc: U102.2 (LPWM)
- new net VDD: J104.1 (Pin_1), JP101.3 (B), JP103.1 (A), U103.1 (IN)
- new net Vout: J101.1 (Pin_1), J105.1 (Pin_1), JP101.2 (C)
- no-connect marks 0 -> 4
Other:
- added sheet HLBlockerH (hlblocker.kicad_sch)
- added sheet HLBlockerL (hlblocker.kicad_sch)
- added sheet JKBlockerJ (jkblocker.kicad_sch)
- added sheet JKBlockerK (jkblocker.kicad_sch)
- added sheet OSD0 (optionalStepDown.kicad_sch)
- added sheet OSD1 (optionalStepDown.kicad_sch)
- added sheet OSD2 (optionalStepDown.kicad_sch)
- added sheet OSD3 (optionalStepDown.kicad_sch)
- note added: "5V Rail Regulator"
- note added: "Blocker Unit"
- note added: "Compute Block"
- note added: "Conditionally pass/block signals based on internal and external factors Final step before signal reaches motor controller"
- note added: "Generate 5V from +12V Remove and bypass if running on +6V battery, due to minimum working voltage of LM7805 regulator If using MCU: NO BYPASS"
- note added: "Includes input signal attenuation (if required)"
- note added: "Input Block"
- note added: "Motor Controllers"
- note added: "Power AUX Output Port"
- note added: "Power Input Port"
- note added: "Power Selection"
- note added: "Select main power rail distributed throughout power bus"
- note added: "Space for a Seeeduino XIAO-family MCU Enables possible on-board processing, if desired (If you see this Dr. Santos... pretend you didn't)"
