File: GBG_Motors.kicad_sch (KiCad schematic)
At the start: 0 parts

Commit message: Fixed critical missing files
Parts:
- added J101: Input, Connector_PinHeader_2.54mm:PinHeader_1x06_P2.54mm_Vertical, symbol Connector:Conn_01x06_Pin
- added J102: Seeed XIAO L, Connector_PinHeader_2.54mm:PinHeader_1x07_P2.54mm_Vertical, symbol Connector:Conn_01x07_Pin
- added J103: Seeed XIAO R, Connector_PinHeader_2.54mm:PinHeader_1x07_P2.54mm_Vertical, symbol Connector:Conn_01x07_Pin
- added J104: Pin, Connector_PinHeader_2.54mm:PinHeader_1x02_P2.54mm_Vertical, symbol Connector:Conn_01x02_Pin
- added J105: Pout, Connector_PinHeader_2.54mm:PinHeader_1x02_P2.54mm_Vertical, symbol Connector:Conn_01x02_Pin
- added JP101: Input Vcc Sel, Jumper:SolderJumper-3_P1.3mm_Bridged12_RoundedPad1.0x1.5mm, symbol Jumper:SolderJumper_3_Bridged12
- added JP103: Regulator Bypass, Jumper:SolderJumper-2_P1.3mm_Bridged_RoundedPad1.0x1.5mm, symbol Jumper:Jumper_2_Open
- added U101: JK Controller, BTS7960:BTS7960, symbol BTS7960:BTS7960
- added U102: HL Controller, BTS7960:BTS7960, symbol BTS7960:BTS7960
- added U103: R-78E5.0-0.5, Converter_DCDC:Converter_DCDC_RECOM_R-78E-0.5_THT, symbol Converter_DCDC:R-78E5.0-0.5
Connections:
- new net +5V: J103.1 (Pin_1), JP101.1 (A), JP103.2 (B), U101.3 (R_EN), U101.4 (L_EN), U101.7 (Vcc), U102.3 (R_EN), U102.4 (L_EN), U102.7 (Vcc), U103.3 (OUT)
- new net GND: J101.6 (Pin_6), J103.2 (Pin_2), J104.2 (Pin_2), J105.2 (Pin_2), U101.8 (GND), U102.8 (GND), U103.2 (GND)
- new net H: J101.2 (Pin_2)
- new net HRi: J102.2 (Pin_2)
- new net HRo: J102.1 (Pin_1)
- new net Hc: U102.1 (RPWM)
- new net J: J101.3 (Pin_3)
- new net JRi: J102.4 (Pin_4)
- new net JRo: J102.3 (Pin_3)
- new net Jc: U101.2 (LPWM)
- new net K: J101.4 (Pin_4)
- new net KRi: J102.6 (Pin_6)
- new net KRo: J102.5 (Pin_5)
- new net Kc: U101.1 (RPWM)
- new net L: J101.5 (Pin_5)
- new net LRi: J103.5 (Pin_5)
- new net LRo: J103.6 (Pin_6)
- new net Lc: U102.2 (LPWM)
- new net VDD: J104.1 (Pin_1), JP101.3 (B), JP103.1 (A), U103.1 (IN)
- new net Vout: J101.1 (Pin_1), J105.1 (Pin_1), JP101.2 (C)
- no-connect marks 0 -> 4
Other:
- added sheet HLBlockerH (hlblocker.kicad_sch)
- added sheet HLBlockerL (hlblocker.kicad_sch)
- added sheet JKBlockerJ (jkblocker.kicad_sch)
- added sheet JKBlockerK (jkblocker.kicad_sch)
- added sheet OSD0 (optionalStepDown.kicad_sch)
- added sheet OSD1 (optionalStepDown.kicad_sch)
- added sheet OSD2 (optionalStepDown.kicad_sch)
- added sheet OSD3 (optionalStepDown.kicad_sch)
- note added: "5V Rail Regulator"
- note added: "Blocker Unit"
- note added: "Compute Block"
- note added: "Conditionally pass/block signals based on internal and external factors Final step before signal reaches motor controller"
- note added: "Generate 5V from +12V Remove and bypass if running on +6V battery, due to minimum working voltage of LM7805 regulator If using MCU: NO BYPASS"
- note added: "Includes input signal attenuation (if required)"
- note added: "Input Block"
- note added: "Motor Controllers"
- note added: "Power AUX Output Port"
- note added: "Power Input Port"
- note added: "Power Selection"
- note added: "Select main power rail distributed throughout power bus"
- note added: "Space for a Seeeduino XIAO-family MCU Enables possible on-board processing, if desired (If you see this Dr. Santos... pretend you didn't)"

Commit message: Finished initial board design
Parts:
- JP103: footprint Jumper:SolderJumper-2_P1.3mm_Bridged_RoundedPad1.0x1.5mm -> Jumper:SolderJumper-2_P1.3mm_Open_RoundedPad1.0x1.5mm
Changed lines of the file:
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@@
 			)
 		)
-		(property "Footprint" "Jumper:SolderJumper-2_P1.3mm_Bridged_RoundedPad1.0x1.5mm"
+		(property "Footprint" "Jumper:SolderJumper-2_P1.3mm_Open_RoundedPad1.0x1.5mm"
 			(at 127 27.94 0)
 			(hide yes)

Commit message: Replaced VDD/5V passthru with fully-fledged pin header
Parts:
- removed JP103: Regulator Bypass, Jumper:SolderJumper-2_P1.3mm_Open_RoundedPad1.0x1.5mm, symbol Jumper:Jumper_2_Open
- added J106: Bypass, Connector_PinSocket_2.54mm:PinSocket_1x03_P2.54mm_Vertical, symbol Connector:Conn_01x03_Pin
Connections:
- net +5V: now also J106.1 (Pin_1)
- net VDD: now also J106.2 (Pin_2)
- no-connect marks 4 -> 5
Changed lines of the file:
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@@
 	)
 	(junction
-		(at 137.16 27.94)
+		(at 137.16 33.02)
 		(diameter 0)
 		(color 0 0 0 0)
@@
 	)
 	(junction
-		(at 116.84 27.94)
+		(at 116.84 33.02)
 		(diameter 0)
 		(color 0 0 0 0)
@@
 	)
 	(no_connect
+		(at 124.46 30.48)
+	)
+	(no_connect
 		(at 181.61 35.56)
 	)
@@
 	(wire
 		(pts
-			(xy 137.16 25.4) (xy 137.16 27.94)
-		)
-		(stroke
-			(width 0)
-			(type default)
-		)
-	)
-	(wire
-		(pts
 			(xy 58.42 85.09) (xy 55.88 85.09)
 		)
@@
 	(wire
 		(pts
-			(xy 116.84 27.94) (xy 116.84 25.4)
+			(xy 116.84 25.4) (xy 116.84 33.02)
 		)
 		(stroke
@@
 	(wire
 		(pts
-			(xy 116.84 27.94) (xy 121.92 27.94)
-		)
-		(stroke
-			(width 0)
-			(type default)
-		)
-	)
-	(wire
-		(pts
 			(xy 153.67 74.93) (xy 156.21 74.93)
 		)
@@
 	(wire
 		(pts
+			(xy 116.84 33.02) (xy 127 33.02)
+		)
+		(stroke
+			(width 0)
+			(type default)
+		)
+	)
+	(wire
+		(pts
 			(xy 215.9 95.25) (xy 218.44 95.25)
 		)
@@
 	(wire
 		(pts
-			(xy 158.75 45.72) (xy 147.32 45.72)
+			(xy 129.54 30.48) (xy 129.54 33.02)
 		)
 		(stroke
@@
 	(wire
 		(pts
-			(xy 153.67 100.33) (xy 156.21 100.33)
+			(xy 127 33.02) (xy 127 30.48)
 		)
 		(stroke
@@
 	(wire
 		(pts
-			(xy 180.34 134.62) (xy 184.15 134.62)
+			(xy 158.75 45.72) (xy 147.32 45.72)
 		)
 		(stroke
@@
 	(wire
 		(pts
-			(xy 153.67 82.55) (xy 156.21 82.55)
+			(xy 153.67 100.33) (xy 156.21 100.33)
 		)
 		(stroke
@@
 	(wire
 		(pts
-			(xy 186.69 27.94) (xy 186.69 43.18)
+			(xy 180.34 134.62) (xy 184.15 134.62)
 		)
 		(stroke
@@
 	(wire
 		(pts
-			(xy 95.25 46.99) (xy 97.79 46.99)
+			(xy 153.67 82.55) (xy 156.21 82.55)
 		)
 		(stroke
@@
 	(wire
 		(pts
-			(xy 176.53 95.25) (xy 179.07 95.25)
+			(xy 186.69 27.94) (xy 186.69 43.18)
 		)
 		(stroke
@@
 	(wire
 		(pts
-			(xy 57.15 49.53) (xy 57.15 46.99)
+			(xy 95.25 46.99) (xy 97.79 46.99)
 		)
 		(stroke
@@
 	(wire
 		(pts
-			(xy 116.84 45.72) (xy 116.84 27.94)
+			(xy 176.53 95.25) (xy 179.07 95.25)
+		)
+		(stroke
+			(width 0)
+			(type default)
+		)
+	)
+	(wire
+		(pts
+			(xy 57.15 49.53) (xy 57.15 46.99)
 		)
 		(stroke
@@
 	(wire
 		(pts
+			(xy 137.16 33.02) (xy 137.16 45.72)
+		)
+		(stroke
+			(width 0)
+			(type default)
+		)
+	)
+	(wire
+		(pts
 			(xy 58.42 87.63) (xy 55.88 87.63)
 		)
@@
 	(wire
 		(pts
-			(xy 132.08 27.94) (xy 137.16 27.94)
+			(xy 186.69 43.18) (xy 196.85 43.18)
 		)
 		(stroke
@@
 	(wire
 		(pts
-			(xy 186.69 43.18) (xy 196.85 43.18)
+			(xy 105.41 88.9) (xy 105.41 91.44)
 		)
 		(stroke
@@
 	(wire
 		(pts
-			(xy 105.41 88.9) (xy 105.41 91.44)
+			(xy 102.87 88.9) (xy 105.41 88.9)
 		)
 		(stroke
@@
 	(wire
 		(pts
-			(xy 102.87 88.9) (xy 105.41 88.9)
+			(xy 127 55.88) (xy 127 53.34)
 		)
 		(stroke
@@
 	(wire
 		(pts
-			(xy 127 55.88) (xy 127 53.34)
+			(xy 73.66 24.13) (xy 76.2 24.13)
 		)
 		(stroke
@@
 	(wire
 		(pts
-			(xy 73.66 24.13) (xy 76.2 24.13)
+			(xy 116.84 33.02) (xy 116.84 45.72)
 		)
 		(stroke
@@
 	(wire
 		(pts
+			(xy 129.54 33.02) (xy 137.16 33.02)
+		)
+		(stroke
+			(width 0)
+			(type default)
+		)
+	)
+	(wire
+		(pts
 			(xy 196.85 137.16) (xy 196.85 139.7)
 		)
@@
 	(wire
 		(pts
-			(xy 137.16 27.94) (xy 137.16 45.72)
+			(xy 137.16 25.4) (xy 137.16 33.02)
 		)
 		(stroke
@@
 	)
 	(symbol
+		(lib_id "Connector:Conn_01x03_Pin")
+		(at 127 25.4 270)
+		(unit 1)
+		(body_style 1)
+		(exclude_from_sim no)
+		(in_bom yes)
+		(on_board yes)
+		(in_pos_files yes)
+		(dnp no)
+		(fields_autoplaced yes)
+		(property "Reference" "J106"
+			(at 127 20.32 90)
+			(show_name no)
+			(do_not_autoplace no)
+			(effects
+				(font
+					(size 1.27 1.27)
+				)
+			)
+		)
+		(property "Value" "Bypass"
+			(at 127 22.86 90)
+			(show_name no)
+			(do_not_autoplace no)
+			(effects
+				(font
+					(size 1.27 1.27)
+				)
+			)
+		)
+		(property "Footprint" "Connector_PinSocket_2.54mm:PinSocket_1x03_P2.54mm_Vertical"
+			(at 127 25.4 0)
+			(hide yes)
+			(show_name no)
+			(do_not_autoplace no)
+			(effects
+				(font
+					(size 1.27 1.27)
+				)
+			)
+		)
+		(property "Datasheet" ""
+			(at 127 25.4 0)
+			(hide yes)
+			(show_name no)
+			(do_not_autoplace no)
+			(effects
+				(font
+					(size 1.27 1.27)
+				)
+			)
+		)
+		(property "Description" "Generic connector, single row, 01x03, script generated"
+			(at 127 25.4 0)
+			(hide yes)
+			(show_name no)
+			(do_not_autoplace no)
+			(effects
+				(font
+					(size 1.27 1.27)
+				)
+			)
+		)
+		(pin "1"
+		)
+		(pin "2"
+		)
+		(pin "3"
+		)
+		(instances
+			(project "GBG_Motors"
+				(path "/e3f71057-02b7-45a4-9125-5183de1d436b"
+					(reference "J106")
+					(unit 1)
+				)
+			)
+		)
+	)
+	(symbol
 		(lib_id "power:GND")
 		(at 170.18 54.61 0)
@@
 					(unit 1)
 				)
-			)
-		)
-	)
-	(symbol
-		(lib_id "Jumper:Jumper_2_Open")
-		(at 127 27.94 0)
-		(unit 1)
-		(body_style 1)
-		(exclude_from_sim no)
-		(in_bom yes)
-		(on_board yes)
-		(in_pos_files yes)
-		(dnp no)
-		(fields_autoplaced yes)
-		(property "Reference" "JP103"
-			(at 127 21.59 0)
-			(show_name no)
-			(do_not_autoplace no)
-			(effects
-				(font
-					(size 1.27 1.27)
-				)
-			)
-		)
-		(property "Value" "Regulator Bypass"
-			(at 127 24.13 0)
-			(show_name no)
-			(do_not_autoplace no)
-			(effects
-				(font
-					(size 1.27 1.27)
-				)
-			)
-		)
-		(property "Footprint" "Jumper:SolderJumper-2_P1.3mm_Open_RoundedPad1.0x1.5mm"
-			(at 127 27.94 0)
-			(hide yes)
-			(show_name no)
-			(do_not_autoplace no)
-			(effects
-				(font
-					(size 1.27 1.27)
-				)
-			)
-		)
-		(property "Datasheet" ""
-			(at 127 27.94 0)
-			(hide yes)
-			(show_name no)
-			(do_not_autoplace no)
-			(effects
-				(font
-					(size 1.27 1.27)
-				)
-			)
-		)
-		(property "Description" "Jumper, 2-pole, open"
-			(at 127 27.94 0)
-			(hide yes)
-			(show_name no)
-			(do_not_autoplace no)
-			(effects
-				(font
-					(size 1.27 1.27)
-				)
-			)
-		)
-		(pin "2"
-		)
-		(pin "1"
-		)
-		(instances
-			(project "GBG_Motors"
-				(path "/e3f71057-02b7-45a4-9125-5183de1d436b"
-					(reference "JP103")
-					(unit 1)
-				)

Commit message: Updated bypass jumper pin header model
Parts:
- J106: footprint Connector_PinSocket_2.54mm:PinSocket_1x03_P2.54mm_Vertical -> Connector_PinHeader_2.54mm:PinHeader_1x03_P2.54mm_Vertical
Changed lines of the file:
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@@
 			)
 		)
-		(property "Footprint" "Connector_PinSocket_2.54mm:PinSocket_1x03_P2.54mm_Vertical"
+		(property "Footprint" "Connector_PinHeader_2.54mm:PinHeader_1x03_P2.54mm_Vertical"
 			(at 127 25.4 0)
 			(hide yes)

Commit message: Added bypass capacitor
Parts:
- removed U103: R-78E5.0-0.5, Converter_DCDC:Converter_DCDC_RECOM_R-78E-0.5_THT, symbol Converter_DCDC:R-78E5.0-0.5
- added C102: 0.22uF, Capacitor_THT:C_Axial_L3.8mm_D2.6mm_P7.50mm_Horizontal, symbol Device:C
- added U103: LM7805_TO220, Package_TO_SOT_THT:TO-220-3_Vertical, symbol Regulator_Linear:LM7805_TO220
Connections:
- net +5V: now also J106.2 (Pin_2); no longer J106.1 (Pin_1)
- net GND: now also C102.2, U103.2 (GND)
- net VDD: now also J106.1 (Pin_1), C102.1, U103.1 (VI); no longer J106.2 (Pin_2)
- net at J106.3 (Pin_3): now also U103.3 (VO)
- no-connect marks 5 -> 4
Other:
- note added: "Max Vcc limited by SN74HC244 buffer 7V MAX"
- moved on the sheet: J106
