File: jkblocker.kicad_sch (KiCad schematic)
At the start: 2 parts

Commit message: Finished initial board design
Parts:
- renumbered JP802 to JP801, JP803 to JP802
Changed lines of the file:
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@@
 		(in_pos_files yes)
 		(dnp no)
-		(property "Reference" "JP803"
+		(property "Reference" "JP802"
 			(at 156.21 105.4099 90)
 			(show_name no)
@@
 				)
 				(path "/e3f71057-02b7-45a4-9125-5183de1d436b/e09b614a-aee1-4e93-a129-1f0bfe5e2d84"
-					(reference "JP803")
+					(reference "JP802")
 					(unit 1)
 				)
@@
 		(in_pos_files yes)
 		(dnp no)
-		(property "Reference" "JP802"
+		(property "Reference" "JP801"
 			(at 133.35 105.41 90)
 			(show_name no)
@@
 				)
 				(path "/e3f71057-02b7-45a4-9125-5183de1d436b/e09b614a-aee1-4e93-a129-1f0bfe5e2d84"
-					(reference "JP802")
+					(reference "JP801")
 					(unit 1)
 				)
