File: hlblocker.kicad_sch (KiCad schematic)
At the start: 14 parts, among them J601 Limit Switch, Q602 NPN, U601 NE555P

Commit message: Finished initial board design
Parts:
- renumbered JP602 to JP601, JP601 to JP602, Q602 to Q601, R607 to R605, R605 to R607
Changed lines of the file:
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@@
 		(in_pos_files yes)
 		(dnp no)
-		(property "Reference" "R607"
+		(property "Reference" "R605"
 			(at 118.618 38.1 0)
 			(show_name no)
@@
 				)
 				(path "/e3f71057-02b7-45a4-9125-5183de1d436b/7b5dadd4-4dea-49c5-be78-f4ebd2518203"
-					(reference "R607")
+					(reference "R605")
 					(unit 1)
 				)
@@
 		(dnp no)
 		(fields_autoplaced yes)
-		(property "Reference" "Q602"
+		(property "Reference" "Q601"
 			(at 123.19 71.1199 0)
 			(show_name no)
@@
 				)
 				(path "/e3f71057-02b7-45a4-9125-5183de1d436b/7b5dadd4-4dea-49c5-be78-f4ebd2518203"
-					(reference "Q602")
+					(reference "Q601")
 					(unit 1)
 				)
@@
 		(dnp no)
 		(fields_autoplaced yes)
-		(property "Reference" "JP602"
+		(property "Reference" "JP601"
 			(at 46.99 59.69 0)
 			(show_name no)
@@
 				)
 				(path "/e3f71057-02b7-45a4-9125-5183de1d436b/7b5dadd4-4dea-49c5-be78-f4ebd2518203"
-					(reference "JP602")
+					(reference "JP601")
 					(unit 1)
 				)
@@
 		(in_pos_files yes)
 		(dnp no)
-		(property "Reference" "JP601"
+		(property "Reference" "JP602"
 			(at 74.93 64.77 0)
 			(show_name no)
@@
 				)
 				(path "/e3f71057-02b7-45a4-9125-5183de1d436b/7b5dadd4-4dea-49c5-be78-f4ebd2518203"
-					(reference "JP601")
+					(reference "JP602")
 					(unit 1)
 				)
@@
 		(dnp no)
 		(fields_autoplaced yes)
-		(property "Reference" "R605"
+		(property "Reference" "R607"
 			(at 129.54 35.5599 0)
 			(show_name no)
@@
 				)
 				(path "/e3f71057-02b7-45a4-9125-5183de1d436b/7b5dadd4-4dea-49c5-be78-f4ebd2518203"
-					(reference "R605")
-					(unit 1)
-				)
+					(reference "R607")
+					(unit 1)
+				)

Commit message: Final changes based on BoM
Parts:
- removed R602: 10k, Resistor_THT:R_Axial_DIN0207_L6.3mm_D2.5mm_P7.62mm_Horizontal, symbol Device:R_US
- R601: value R -> 10k
Changed lines of the file:
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@@
-	)
-	(junction
-		(at 87.63 72.39)
-		(diameter 0)
-		(color 0 0 0 0)
 	)
 	(junction
@@
 	(wire
 		(pts
-			(xy 87.63 72.39) (xy 90.17 72.39)
-		)
-		(stroke
-			(width 0)
-			(type default)
-		)
-	)
-	(wire
-		(pts
 			(xy 120.65 40.64) (xy 120.65 64.77)
 		)
@@
 	(wire
 		(pts
-			(xy 87.63 74.93) (xy 87.63 72.39)
-		)
-		(stroke
-			(width 0)
-			(type default)
-		)
-	)
-	(wire
-		(pts
 			(xy 120.65 64.77) (xy 120.65 67.31)
 		)
@@
 	(wire
 		(pts
-			(xy 71.12 72.39) (xy 87.63 72.39)
+			(xy 71.12 72.39) (xy 90.17 72.39)
 		)
 		(stroke
@@
 		(pts
 			(xy 186.69 69.85) (xy 186.69 101.6)
-		)
-		(stroke
-			(width 0)
-			(type default)
-		)
-	)
-	(wire
-		(pts
-			(xy 87.63 82.55) (xy 87.63 85.09)
 		)
 		(stroke
@@
 	)
 	(symbol
-		(lib_id "power:GND")
-		(at 87.63 85.09 0)
-		(unit 1)
-		(body_style 1)
-		(exclude_from_sim no)
-		(in_bom yes)
-		(on_board yes)
-		(in_pos_files yes)
-		(dnp no)
-		(fields_autoplaced yes)
-		(property "Reference" "#PWR0603"
-			(at 87.63 91.44 0)
-			(hide yes)
-			(show_name no)
-			(do_not_autoplace no)
-			(effects
-				(font
-					(size 1.27 1.27)
-				)
-			)
-		)
-		(property "Value" "GND"
-			(at 87.63 90.17 0)
-			(show_name no)
-			(do_not_autoplace no)
-			(effects
-				(font
-					(size 1.27 1.27)
-				)
-			)
-		)
-		(property "Footprint" ""
-			(at 87.63 85.09 0)
-			(hide yes)
-			(show_name no)
-			(do_not_autoplace no)
-			(effects
-				(font
-					(size 1.27 1.27)
-				)
-			)
-		)
-		(property "Datasheet" ""
-			(at 87.63 85.09 0)
-			(hide yes)
-			(show_name no)
-			(do_not_autoplace no)
-			(effects
-				(font
-					(size 1.27 1.27)
-				)
-			)
-		)
-		(property "Description" "Power symbol creates a global label with name \"GND\" , ground"
-			(at 87.63 85.09 0)
-			(hide yes)
-			(show_name no)
-			(do_not_autoplace no)
-			(effects
-				(font
-					(size 1.27 1.27)
-				)
-			)
-		)
-		(pin "1"
-		)
-		(instances
-			(project "GBG_Motors"
-				(path "/e3f71057-02b7-45a4-9125-5183de1d436b/29ea8377-c72d-49b7-85fa-ba09c5d0bc93"
-					(reference "#PWR0702")
-					(unit 1)
-				)
-				(path "/e3f71057-02b7-45a4-9125-5183de1d436b/7b5dadd4-4dea-49c5-be78-f4ebd2518203"
-					(reference "#PWR0603")
-					(unit 1)
-				)
-			)
-		)
-	)
-	(symbol
 		(lib_id "Device:R")
 		(at 59.69 71.12 0)
@@
 			)
 		)
-		(property "Value" "R"
+		(property "Value" "10k"
 			(at 62.23 72.3899 0)
 			(show_name no)
@@
 		)
 		(property "Value" "redirect"
-			(at 77.47 64.77 0)
+			(at 77.47 64.77 90)
 			(show_name no)
 			(do_not_autoplace no)
@@
 					(unit 1)
 				)
-			)
-		)
-	)
-	(symbol
-		(lib_id "Device:R_US")
-		(at 87.63 78.74 0)
-		(unit 1)
-		(body_style 1)
-		(exclude_from_sim no)
-		(in_bom yes)
-		(on_board yes)
-		(in_pos_files yes)
-		(dnp no)
-		(fields_autoplaced yes)
-		(property "Reference" "R602"
-			(at 90.17 77.4699 0)
-			(show_name no)
-			(do_not_autoplace no)
-			(effects
-				(font
-					(size 1.27 1.27)
-				)
-				(justify left)
-			)
-		)
-		(property "Value" "10k"
-			(at 90.17 80.0099 0)
-			(show_name no)
-			(do_not_autoplace no)
-			(effects
-				(font
-					(size 1.27 1.27)
-				)
-				(justify left)
-			)
-		)
-		(property "Footprint" "Resistor_THT:R_Axial_DIN0207_L6.3mm_D2.5mm_P7.62mm_Horizontal"
-			(at 88.646 78.994 90)
-			(hide yes)
-			(show_name no)
-			(do_not_autoplace no)
-			(effects
-				(font
-					(size 1.27 1.27)
-				)
-			)
-		)
-		(property "Datasheet" ""
-			(at 87.63 78.74 0)
-			(hide yes)
-			(show_name no)
-			(do_not_autoplace no)
-			(effects
-				(font
-					(size 1.27 1.27)
-				)
-			)
-		)
-		(property "Description" "Resistor, US symbol"
-			(at 87.63 78.74 0)
-			(hide yes)
-			(show_name no)
-			(do_not_autoplace no)
-			(effects
-				(font
-					(size 1.27 1.27)
-				)
-			)
-		)
-		(pin "1"
-		)
-		(pin "2"
-		)
-		(instances
-			(project "GBG_Motors"
-				(path "/e3f71057-02b7-45a4-9125-5183de1d436b/29ea8377-c72d-49b7-85fa-ba09c5d0bc93"
-					(reference "R702")
-					(unit 1)
-				)
-				(path "/e3f71057-02b7-45a4-9125-5183de1d436b/7b5dadd4-4dea-49c5-be78-f4ebd2518203"
-					(reference "R602")
-					(unit 1)
-				)
